File: sram-breadboard-adaptor.kicad_pcb (KiCad board)
At the start: 4 copper layers, 121.9 x 45.7 mm, 20 parts, among them J0 Conn_01x40, J1 Conn_01x40, U0 LY62W10248ML-55LLI, U1 LY62W10248ML-55LLI, U2 LY62W10248ML-55LLI, U3 LY62W10248ML-55LLI, U4 LY62W10248ML-55LLI, U5 LY62W10248ML-55LLI, U6 LY62W10248ML-55LLI, U7 LY62W10248ML-55LLI

Commit message: v1.0 candidate
Parts:
- moved C7 0.68 mm to (210.1, 65.5)
- moved C5 0.67 mm to (180.8, 65.5)
- moved C4 0.67 mm to (166.1, 65.5)
- moved C3 0.67 mm to (151.4, 65.5)
- moved C6 0.67 mm to (195.6, 65.5)
- moved C1 0.48 mm to (121.9, 65.5)
- moved C0 0.47 mm to (107.2, 65.5)
- moved C2 0.47 mm to (136.6, 65.5)
- renumbered U0 to A0, U1 to A1, U2 to A2, U3 to A3, U4 to B0, U5 to B1, U6 to B2, U7 to B3
Routing:
- net /D25: track 93.9 -> 91.6 mm
- net /A5: track 171.7 -> 169.4 mm
- net /D24: track 91.6 -> 89.4 mm
- net /D27: track 101.8 -> 99.7 mm
- net /A18: track 134.7 -> 136.8 mm
- net /D28: track 102.2 -> 100.2 mm
- net /D20: track 101.7 -> 99.7 mm
- net /D26: track 99.4 -> 97.4 mm
- net /D15: track 103.9 -> 105.4 mm
- net /D29: track 101.3 -> 99.9 mm
- net /D14: track 105.3 -> 106.7 mm
- net /D23: track 95.0 -> 96.3 mm
- net /D19: track 100.5 -> 99.3 mm
- net /D18: track 98.0 -> 96.9 mm
- net /~{CEA2}: track 76.6 -> 77.6 mm
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Other:
- board text added: "100nF"
- board text added: "330R"
- board text added: "R/~{W}"
- board text added: "VCC"
- board text added: "http://github.com/sparkybrit/sram-breadboard-adaptor (c) 2023 Graeme Harker v1.0"
- board text removed: "+5V"
- board text removed: "R~{W}"
- board text removed: "http://sparkybrit/sram-breadboard-adaptor v1.0 (c) 2023 Graeme Harker"
- board text removed: "sram-breadboard-adaptor V1.0.0 (c) 2023 Graeme Harker"
